File: hardware/vendotron_v1.brd (EAGLE design)
At the start: 60 x 80 mm, 22 parts, among them J5 POWER_JACKPTH

Commit message: Updates
Connections:
- new net EN_N: U$1.8, U$2.EN_N
Routing:
- net EN_N: track 0.00 -> 41.0 mm, vias 0 -> 1
- net SERVO4: track 72.1 -> 69.6 mm
- net 5V: track 159.5 -> 160.9 mm
- net SERVO5: track 77.5 -> 76.3 mm
- net SERVO2: track 61.5 -> 62.3 mm
Other:
- board text added: "Vendotron"
- board text removed: "Vendotron 5000"
Changed lines of the file:
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@@
 <hole x="55" y="5" drill="3.2"/>
 <hole x="19" y="27" drill="3.2"/>
-<text x="7.6" y="62" size="2.54" layer="21" font="vector" rot="R90" align="center">Vendotron
-5000</text>
+<text x="7.6" y="62" size="2.54" layer="21" font="vector" rot="R90" align="center">Vendotron</text>
 <text x="48" y="2" size="1.778" layer="21">v1</text>
 <text x="52" y="43" size="1.27" layer="21" rot="R90">LEDS</text>
@@
 <wire x1="47" y1="30" x2="43.92" y2="30" width="0.4064" layer="16"/>
 <wire x1="43.92" y1="30" x2="31.65" y2="17.73" width="0.4064" layer="16"/>
+<wire x1="7" y1="23" x2="6" y2="24" width="0.4064" layer="16"/>
 </signal>
 <signal name="VIN">
@@
 <wire x1="10" y1="32" x2="46" y2="32" width="0.4064" layer="16"/>
 <wire x1="46" y1="32" x2="52" y2="38" width="0.4064" layer="16"/>
-<wire x1="52" y1="38" x2="52" y2="54" width="0.4064" layer="16"/>
-<wire x1="52" y1="54" x2="50" y2="56" width="0.4064" layer="16"/>
-<wire x1="50" y1="56" x2="38.932" y2="56" width="0.4064" layer="16"/>
+<wire x1="52" y1="38" x2="52" y2="52" width="0.4064" layer="16"/>
+<wire x1="52" y1="52" x2="48" y2="56" width="0.4064" layer="16"/>
+<wire x1="48" y1="56" x2="38.932" y2="56" width="0.4064" layer="16"/>
 <wire x1="38.932" y1="56" x2="38.68" y2="55.748" width="0.4064" layer="16"/>
 </signal>
@@
 <wire x1="8.08" y1="34" x2="46" y2="34" width="0.4064" layer="16"/>
 <wire x1="46" y1="34" x2="51" y2="39" width="0.4064" layer="16"/>
-<wire x1="51" y1="39" x2="51" y2="53" width="0.4064" layer="16"/>
-<wire x1="51" y1="53" x2="50" y2="54" width="0.4064" layer="16"/>
-<wire x1="50" y1="54" x2="39.472" y2="54" width="0.4064" layer="16"/>
-<wire x1="39.472" y1="54" x2="38.68" y2="53.208" width="0.4064" layer="16"/>
+<wire x1="51" y1="39" x2="51" y2="50" width="0.4064" layer="16"/>
+<wire x1="51" y1="50" x2="48" y2="53" width="0.4064" layer="16"/>
+<wire x1="48" y1="53" x2="39.472" y2="53" width="0.4064" layer="16"/>
+<wire x1="39.472" y1="53" x2="38.68" y2="53.208" width="0.4064" layer="16"/>
 </signal>
 <signal name="SERVO3">
@@
 <contactref element="S3" pad="3"/>
 <wire x1="8.08" y1="38" x2="8.08" y2="36.92" width="0.4064" layer="16"/>
-<wire x1="8.08" y1="36.92" x2="9" y2="36" width="0.4064" layer="16"/>
-<wire x1="9" y1="36" x2="46" y2="36" width="0.4064" layer="16"/>
-<wire x1="46" y1="36" x2="50" y2="40" width="0.4064" layer="16"/>
-<wire x1="50" y1="40" x2="50" y2="50" width="0.4064" layer="16"/>
-<wire x1="50" y1="50" x2="49" y2="51" width="0.4064" layer="16"/>
-<wire x1="49" y1="51" x2="39.012" y2="51" width="0.4064" layer="16"/>
+<wire x1="8.08" y1="36.92" x2="10" y2="35" width="0.4064" layer="16"/>
+<wire x1="10" y1="35" x2="45" y2="35" width="0.4064" layer="16"/>
+<wire x1="45" y1="35" x2="50" y2="40" width="0.4064" layer="16"/>
+<wire x1="50" y1="40" x2="50" y2="48" width="0.4064" layer="16"/>
+<wire x1="50" y1="48" x2="47" y2="51" width="0.4064" layer="16"/>
+<wire x1="47" y1="51" x2="39.012" y2="51" width="0.4064" layer="16"/>
 <wire x1="39.012" y1="51" x2="38.68" y2="50.668" width="0.4064" layer="16"/>
 </signal>
 <signal name="SERVO2">
 <contactref element="U$1" pad="13"/>
-<wire x1="8.08" y1="40.92" x2="12" y2="37" width="0.4064" layer="16"/>
-<wire x1="12" y1="37" x2="45" y2="37" width="0.4064" layer="16"/>
-<wire x1="45" y1="37" x2="49" y2="41" width="0.4064" layer="16"/>
+<wire x1="8.08" y1="40.92" x2="13" y2="36" width="0.4064" layer="16"/>
+<wire x1="13" y1="36" x2="44" y2="36" width="0.4064" layer="16"/>
+<wire x1="44" y1="36" x2="49" y2="41" width="0.4064" layer="16"/>
 <wire x1="49" y1="41" x2="49" y2="46" width="0.4064" layer="16"/>
-<wire x1="49" y1="46" x2="46.952" y2="48.1" width="0.4064" layer="16"/>
-<wire x1="46.952" y1="48.1" x2="38.68" y2="48.128" width="0.4064" layer="16"/>
+<wire x1="49" y1="46" x2="47" y2="48" width="0.4064" layer="16"/>
 <contactref element="S2" pad="3"/>
 <wire x1="8.08" y1="40.92" x2="8.08" y2="42" width="0.6096" layer="16"/>
+<wire x1="47" y1="48" x2="38.808" y2="48" width="0.4064" layer="16"/>
+<wire x1="38.808" y1="48" x2="38.68" y2="48.128" width="0.4064" layer="16"/>
 </signal>
 <signal name="STEP_N">
@@
 <wire x1="26.698" y1="22.81" x2="26.508" y2="23" width="0.4064" layer="1"/>
 </signal>
+<signal name="EN_N">
+<contactref element="U$2" pad="EN_N"/>
+<wire x1="31.65" y1="27.89" x2="31.65" y2="28.35" width="0.4064" layer="1"/>
+<wire x1="31.65" y1="28.35" x2="29" y2="31" width="0.4064" layer="1"/>
+<wire x1="29" y1="31" x2="24" y2="31" width="0.4064" layer="1"/>
+<wire x1="24" y1="31" x2="17" y2="38" width="0.4064" layer="1"/>
+<via x="17" y="38" extent="1-16" drill="0.8"/>
+<contactref element="U$1" pad="8"/>
+<wire x1="17" y1="38" x2="17" y2="54.388" width="0.4064" layer="16"/>
+<wire x1="17" y1="54.388" x2="20.9" y2="58.288" width="0.4064" layer="16"/>
+</signal>
 </signals>
