File: hardware/vendotron_v1.sch (EAGLE design)
At the start: 20 parts, among them J5 POWER_JACKPTH

Commit message: Updates
Connections:
- new net EN_N: U$1.A4, U$2.EN_N
Changed lines of the file:
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@@
 <segment>
 <pinref part="U$1" gate="G$1" pin="A0"/>
-<wire x1="0" y1="22.86" x2="-15.24" y2="22.86" width="0.1524" layer="91"/>
-<label x="-15.24" y="22.86" size="1.778" layer="95"/>
+<wire x1="0" y1="22.86" x2="-12.7" y2="22.86" width="0.1524" layer="91"/>
+<label x="-12.7" y="22.86" size="1.778" layer="95"/>
 </segment>
 </net>
@@
 <segment>
 <pinref part="U$1" gate="G$1" pin="A1"/>
-<wire x1="0" y1="27.94" x2="-15.24" y2="27.94" width="0.1524" layer="91"/>
-<label x="-15.24" y="27.94" size="1.778" layer="95"/>
+<wire x1="0" y1="27.94" x2="-12.7" y2="27.94" width="0.1524" layer="91"/>
+<label x="-12.7" y="27.94" size="1.778" layer="95"/>
 </segment>
 <segment>
@@
 <segment>
 <pinref part="U$1" gate="G$1" pin="A2"/>
-<wire x1="0" y1="33.02" x2="-15.24" y2="33.02" width="0.1524" layer="91"/>
-<label x="-15.24" y="33.02" size="1.778" layer="95"/>
+<wire x1="0" y1="33.02" x2="-12.7" y2="33.02" width="0.1524" layer="91"/>
+<label x="-12.7" y="33.02" size="1.778" layer="95"/>
 </segment>
 </net>
@@
 </segment>
 </net>
+<net name="EN_N" class="0">
+<segment>
+<pinref part="U$2" gate="G$1" pin="EN_N"/>
+<wire x1="5.08" y1="-7.62" x2="0" y2="-7.62" width="0.1524" layer="91"/>
+</segment>
+<segment>
+<pinref part="U$1" gate="G$1" pin="A4"/>
+<wire x1="0" y1="43.18" x2="-12.7" y2="43.18" width="0.1524" layer="91"/>
+<label x="-12.7" y="43.18" size="1.778" layer="95"/>
+</segment>
+</net>
